File: zx-specdrum-re-created.kicad_pcb (KiCad board)
At the start: 2 copper layers, 76 x 51.4 mm, 29 parts, among them J1 ZX_Spectrum_Connector_48K, J2 Audio out, U1 74LS32, U2 TL084

Commit message: Version 1.2 update
Parts:
- added J3: Filter, Connector_PinHeader_2.54mm:PinHeader_1x03_P2.54mm_Vertical, F.Cu at (95.1, 101.7)
- C7: value 1uF -> 10uF; footprint Capacitor_THT:C_Disc_D4.3mm_W1.9mm_P5.00mm -> Capacitor_THT:CP_Radial_D5.0mm_P2.50mm
- moved C7 3.59 mm to (161.0, 92.9)
Connections:
- C6 pad 2: Net-(U2D--) -> Net-(J3-Pin_1)
- C7 pad 1: Net-(U2D--) -> Net-(J3-Pin_2)
- U2 pad 13: Net-(U2D--) -> Net-(J3-Pin_1)
- U2 pad 14: Net-(U2D--) -> Net-(J3-Pin_1)
Routing:
- net Net-(J3-Pin_1): track 0.00 -> 83.1 mm
- net Net-(J3-Pin_2): track 0.00 -> 68.6 mm
- net Net-(J3-Pin_3): track 24.4 -> 62.5 mm
- net Net-(U2D--): track 30.0 -> 0.00 mm
- net Net-(U2C-+): track 34.2 -> 45.4 mm
- net ~{IORQ}: track 31.3 -> 38.3 mm, vias 1 -> 0
- net GND: track 194.1 -> 201.0 mm
- net +5V: track 99.2 -> 94.7 mm
- net D1: track 33.6 -> 31.6 mm
- net Net-(C7-Pad2): track 6.01 -> 4.92 mm
Other:
- board text added: "On / Off"
- board text added: "recreated in 2025 v1.2"
- board text removed: "recreated in 2025 v1.1"
