File: zx-specdrum-re-created.kicad_sch (KiCad schematic)
At the start: 28 parts, among them J1 ZX_Spectrum_Connector_48K, J2 Audio out, U1 74LS32, U2 TL084

Commit message: Version 1.2 update
Parts:
- added J3: Filter, Connector_PinHeader_2.54mm:PinHeader_1x03_P2.54mm_Vertical, symbol Connector:Conn_01x03_Pin
- C7: value 1uF -> 10uF; footprint Capacitor_THT:C_Disc_D4.3mm_W1.9mm_P5.00mm -> Capacitor_THT:CP_Radial_D5.0mm_P2.50mm; symbol Device:C -> Device:C_Polarized
Connections:
- net at C6.2, U2.13 (-), U2.14: now also J3.1 (Pin_1); no longer C7.1
- net at R6.1, U2.6 (-), U2.7: now also J3.3 (Pin_3)
- new net: C7.1, J3.2 (Pin_2)
- no-connect marks 42 -> 43
Other:
- moved on the sheet: C9, J2, R10, R11
